File: SPIKE.kicad_pcb (KiCad board)
At the start: 2 copper layers, 29.3 x 56.5 mm, 56 parts, among them J1 Conn_01x17, J2 Conn_01x17, J5 USB_C_Receptacle_USB2.0_14P, SW1 RST, SW2 BOOT, U1 ESP32-S3, U5 TLV62569DRL, U6 APS6404L-3SQRx-SN, U7 W25Q128JVS, Y1 Crystal_GND24

Commit message: Upload gerbers and some modifications
Parts:
- C33: footprint Capacitor_SMD:C_0402_1005Metric -> Capacitor_SMD:C_0603_1608Metric
- L1: footprint Inductor_SMD:L_0201_0603Metric -> Inductor_SMD:L_0603_1608Metric
- L2: footprint Inductor_SMD:L_01005_0402Metric -> Inductor_SMD:L_0201_0603Metric
- R10, R11: footprint Resistor_SMD:R_0805_2012Metric -> Resistor_SMD:R_0603_1608Metric
- R13, R14, R19: footprint Resistor_SMD:R_1206_3216Metric -> Resistor_SMD:R_0603_1608Metric
- moved C10 0.85 mm to (116.4, 85.4), turned to 0 degrees
- moved R14 0.70 mm to (118.1, 102.4)
- moved C6 0.63 mm to (116.5, 89.9)
- moved C33 0.55 mm to (117.0, 87.7)
- moved L2 0.43 mm to (119.5, 85.7)
- moved C34 0.39 mm to (118.4, 88.0)
- moved R19 0.30 mm to (126.2, 82.6)
- moved C5 0.28 mm to (116.4, 94.3)
- moved R13 0.27 mm to (118.1, 100.0)
- moved L1 0.26 mm to (117.0, 92.3)
Routing:
- net GND: track 20.9 -> 19.4 mm, vias 16 -> 17
- net /RST_BTN: track 18.9 -> 20.3 mm
- net 3v3: track 75.2 -> 75.8 mm
