File: SPIKE.kicad_sch (KiCad schematic)
At the start: 54 parts, among them J1 Conn_01x17, J2 Conn_01x17, J5 USB_C_Receptacle_USB2.0_14P, SW1 RST, SW2 BOOT, U1 ESP32-S3, U5 TLV62569DRL, U6 APS6404L-3SQRx-SN, U7 W25Q128JVS, Y1 Crystal_GND24

Commit message: Upload gerbers and some modifications
Parts:
- C33: footprint Capacitor_SMD:C_0402_1005Metric -> Capacitor_SMD:C_0603_1608Metric; MNF PART NUMBER C15195 -> C57112
- L1: footprint Inductor_SMD:L_0201_0603Metric -> Inductor_SMD:L_0603_1608Metric; MNF PART NUMBER C86125 -> C370234
- L2: footprint Inductor_SMD:L_01005_0402Metric -> Inductor_SMD:L_0201_0603Metric; MNF PART NUMBER C74301 -> C139271
- R10, R11: footprint Resistor_SMD:R_0805_2012Metric -> Resistor_SMD:R_0603_1608Metric; MNF PART NUMBER C17561 -> C23345
- R13, R14, R19: footprint Resistor_SMD:R_1206_3216Metric -> Resistor_SMD:R_0603_1608Metric; MNF PART NUMBER C17902 -> C25804
Changed lines of the file:
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@@
 			)
 		)
-		(property "Footprint" "Resistor_SMD:R_0805_2012Metric"
+		(property "Footprint" "Resistor_SMD:R_0603_1608Metric"
 			(at 121.92 108.712 90)
 			(hide yes)
@@
 			)
 		)
-		(property "MNF PART NUMBER" "C17561"
+		(property "MNF PART NUMBER" "C23345"
 			(at 121.92 110.49 0)
 			(hide yes)
@@
 			)
 		)
-		(property "Footprint" "Resistor_SMD:R_1206_3216Metric"
+		(property "Footprint" "Resistor_SMD:R_0603_1608Metric"
 			(at 124.46 164.592 90)
 			(hide yes)
@@
 			)
 		)
-		(property "MNF PART NUMBER" "C17902"
+		(property "MNF PART NUMBER" "C25804"
 			(at 124.46 166.37 0)
 			(hide yes)
@@
 			)
 		)
-		(property "Footprint" "Capacitor_SMD:C_0402_1005Metric"
+		(property "Footprint" "Capacitor_SMD:C_0603_1608Metric"
 			(at 211.7852 49.53 0)
 			(hide yes)
@@
 			)
 		)
-		(property "MNF PART NUMBER" "C15195"
+		(property "MNF PART NUMBER" "C57112"
 			(at 210.82 53.34 0)
 			(hide yes)
@@
 			)
 		)
-		(property "Footprint" "Inductor_SMD:L_01005_0402Metric"
+		(property "Footprint" "Inductor_SMD:L_0201_0603Metric"
 			(at 177.8 139.7 0)
 			(hide yes)
@@
 			)
 		)
-		(property "MNF PART NUMBER" "C74301"
+		(property "MNF PART NUMBER" "C139271"
 			(at 177.8 139.7 90)
 			(hide yes)
@@
 			)
 		)
-		(property "Footprint" "Inductor_SMD:L_0201_0603Metric"
+		(property "Footprint" "Inductor_SMD:L_0603_1608Metric"
 			(at 201.93 22.86 0)
 			(hide yes)
@@
 			)
 		)
-		(property "MNF PART NUMBER" "C86125"
+		(property "MNF PART NUMBER" "C370234"
 			(at 201.93 22.86 90)
 			(hide yes)
@@
 			)
 		)
-		(property "Footprint" "Resistor_SMD:R_0805_2012Metric"
+		(property "Footprint" "Resistor_SMD:R_0603_1608Metric"
 			(at 121.92 106.172 90)
 			(hide yes)
@@
 			)
 		)
-		(property "MNF PART NUMBER" "C17561"
+		(property "MNF PART NUMBER" "C23345"
 			(at 121.92 107.95 0)
 			(hide yes)
@@
 			)
 		)
-		(property "Footprint" "Resistor_SMD:R_1206_3216Metric"
+		(property "Footprint" "Resistor_SMD:R_0603_1608Metric"
 			(at 255.778 36.83 90)
 			(hide yes)
@@
 			)
 		)
-		(property "MNF PART NUMBER" "C17902"
+		(property "MNF PART NUMBER" "C25804"
 			(at 254 36.83 0)
 			(hide yes)
@@
 			)
 		)
-		(property "Footprint" "Resistor_SMD:R_1206_3216Metric"
+		(property "Footprint" "Resistor_SMD:R_0603_1608Metric"
 			(at 281.178 36.83 90)
 			(hide yes)
@@
 			)
 		)
-		(property "MNF PART NUMBER" "C17902"
+		(property "MNF PART NUMBER" "C25804"
 			(at 279.4 36.83 0)
 			(hide yes)
